File: PCB_Joystick/pcb  ag.kicad_pcb (KiCad board)
At the start: 2 copper layers, 80 x 80 mm, 12 parts, among them J2 Conn_01x05, SW10 SW_Push_LED, SW6 SW_Push_LED, SW7 SW_Push_LED, SW8 SW_Push_LED, SW9 SW_Push_LED

Commit message: pcb
Parts:
- added 4.7k1: R, Resistor_SMD:R_0603_1608Metric_Pad0.98x0.95mm_HandSolder, B.Cu at (106.7, 48.2)
- added BT1: Battery, Connector_PinHeader_2.54mm:PinHeader_1x02_P2.54mm_Vertical, B.Cu at (111.5, 85.9)
- added C1: 0.1uF, Capacitor_SMD:C_0603_1608Metric_Pad1.08x0.95mm_HandSolder, B.Cu at (100.4, 76.0)
- added C2: 10uF, Capacitor_SMD:C_0603_1608Metric_Pad1.08x0.95mm_HandSolder, B.Cu at (119.7, 71.3)
- added C3: 0.1uF, Capacitor_SMD:C_0603_1608Metric_Pad1.08x0.95mm_HandSolder, B.Cu at (96.1, 70.5)
- added D6: GREEN, LED_SMD:LED_Cree-XHP50_3V_HighDensity, B.Cu at (106.5, 57.0)
- added D7: RED, LED_SMD:LED_Cree-XHP50_3V_HighDensity, B.Cu at (116.0, 64.3)
- added R10: 1k, Resistor_SMD:R_0603_1608Metric_Pad0.98x0.95mm_HandSolder, B.Cu at (111.5, 80.7)
- added R11: 100, Resistor_SMD:R_0603_1608Metric_Pad0.98x0.95mm_HandSolder, B.Cu at (97.0, 63.3)
- added R12: 1.2k, Resistor_SMD:R_0603_1608Metric_Pad0.98x0.95mm_HandSolder, B.Cu at (106.3, 80.7)
- added R6: 4.7k, Resistor_SMD:R_0603_1608Metric_Pad0.98x0.95mm_HandSolder, B.Cu at (113.2, 47.3)
- added R8: 1k, Resistor_SMD:R_0603_1608Metric_Pad0.98x0.95mm_HandSolder, B.Cu at (101.4, 57.2)
- added R9: 1k, Resistor_SMD:R_0603_1608Metric_Pad0.98x0.95mm_HandSolder, B.Cu at (111.5, 76.0)
- added U2: TP4056-42-ESOP8, footprint:ESOP-8_L4.9-W3.9-P1.27-LS6.0-BL-EP, B.Cu at (106.9, 64.9)
- added U3: FS8205A_C2830320, footprint:SOT-23-6_L2.9-W1.6-P0.95-LS2.8-BR, B.Cu at (113.6, 71.2)
- added U4: DW01A_C351410, footprint:SOT-23-6_L2.9-W1.6-P0.95-LS2.8-BL, B.Cu at (101.3, 70.7)
- added U5: 10155435-00011LF, footprint:USB-C-SMD_10155435-00011LF, F.Cu at (116.5, 55.2)
- R1, R2, R3, R4, R5: footprint Resistor_THT:R_Axial_DIN0207_L6.3mm_D2.5mm_P7.62mm_Horizontal -> Resistor_SMD:R_0603_1608Metric_Pad0.98x0.95mm_HandSolder
- moved U1 154.6 mm to (57.3, 85.9)
- moved R3 32.9 mm to (66.7, 108.0)
- moved SW10 32.1 mm to (61.5, 113.0)
- moved SW7 30.4 mm to (70.0, 57.0), turned to 0 degrees
- moved SW8 29.9 mm to (91.5, 113.0)
- moved R5 29.4 mm to (96.4, 107.8)
- moved R1 26.0 mm to (91.5, 62.9), turned to -90 degrees
- moved R2 18.6 mm to (75.6, 63.0), turned to -90 degrees
- moved SW6 17.3 mm to (86.0, 57.0), turned to 0 degrees
- moved R4 3.98 mm to (81.8, 108.0)
- moved SW9 3.35 mm to (76.5, 113.0)
- moved J2 2.80 mm to (81.5, 80.9)
Routing:
- net GND: track 213.9 -> 375.4 mm, vias 2 -> 11
- net /5button.gpio20: track 97.5 -> 26.5 mm
- net +3V3: track 237.9 -> 168.5 mm, vias 2 -> 0
- net /VBAT+: track 0.00 -> 45.5 mm, vias 0 -> 2
- net Net-(BT1--): track 0.00 -> 41.5 mm, vias 0 -> 4
- net /2button.gpio6: track 49.9 -> 30.5 mm, vias 3 -> 0
- net /3button.gpio7: track 55.0 -> 71.4 mm
- net Net-(U2-~{CHRG}): track 0.00 -> 16.2 mm
- net Net-(U3-G2): track 0.00 -> 16.1 mm, vias 0 -> 2
- net Net-(U5-CC2): track 0.00 -> 15.1 mm, vias 0 -> 1
- net /4button.gpio10: track 53.9 -> 38.9 mm, vias 0 -> 3
- net Net-(U4-VCC): track 0.00 -> 14.5 mm, vias 0 -> 2
- net Net-(D7-K): track 0.00 -> 14.1 mm, vias 0 -> 2
- net Net-(U4-VM): track 0.00 -> 13.1 mm
- net Net-(U2-PROG): track 0.00 -> 13.0 mm
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
Commit message: UPD
Parts:
- D6, D7: footprint LED_SMD:LED_Cree-XHP50_3V_HighDensity -> LED_SMD:LED_0603_1608Metric_Pad1.05x0.95mm_HandSolder
- moved U5 1.29 mm to (117.8, 55.1)
Routing:
- net GND: track 375.4 -> 391.4 mm
- net Net-(U5-CC2): track 15.1 -> 16.7 mm
- net Net-(D7-K): track 14.1 -> 15.4 mm
- net Net-(D6-K): track 10.8 -> 12.0 mm
- net Net-(U5-CC1): track 11.3 -> 12.6 mm
