File: PCB_Main/PCB.kicad_pcb (KiCad board)
At the start: 4 copper layers, 52 x 74.9 mm, 60 parts, among them SW3 SW_Push_Dual, SW4 SW_Push_Dual, U1 RP2350A_C42411118, U2 HDMI-001S, U3 NCP1117-3.3_SOT223, U4 W25Q128JVS, U5 SM03B-SRSS-TB(LF)(SN)(P), U6 10155435-00011LF, U7 Radio Module 2, U8 TLV62569DBVR, X1 TXM12M0004252FBCEO00T

Commit message: upd
Parts:
- added H1: MountingHole, MountingHole:MountingHole_2.5mm, F.Cu at (128.2, 55.0)
- added H2: MountingHole, MountingHole:MountingHole_2.5mm, F.Cu at (84.1, 55.0)
- added H3: MountingHole, MountingHole:MountingHole_2.5mm, F.Cu at (84.1, 121.9)
- added H4: MountingHole, MountingHole:MountingHole_2.5mm, F.Cu at (128.2, 121.9)
Connections:
- net /GPI7 renamed /GPIO7

Commit message: upd
Parts:
- L2, U3: moved to F.Cu
- moved U5 14.9 mm to (92.4, 121.2)
- moved U3 8.31 mm to (111.3, 120.6), turned to 0 degrees
- turned L2 to 0 degrees
Routing:
- net /SWCLK: track 11.1 -> 24.2 mm, vias 0 -> 2
- net VBUS: track 39.1 -> 49.6 mm, vias 2 -> 3
- net /SWD: track 13.2 -> 21.6 mm
- net +3V3: track 68.8 -> 61.2 mm, vias 14 -> 16
- net GND: track 128.1 -> 133.8 mm
- net Net-(U8-SW): track 11.4 -> 16.3 mm, vias 0 -> 1
- net +1V1: track 70.4 -> 73.7 mm, vias 1 -> 2
- net /USB_D-: track 42.6 -> 43.2 mm
