File: PCB_Main/PCB.kicad_sch (KiCad schematic)
At the start: 53 parts, among them Q1 DMG1012T-7, SW1 SW_Push, SW2 SW_Push, U1 RP2350A_C42411118, U2 HDMI-001S, U3 NCP1117-3.3_SOT223, U4 W25Q128JVS, U5 SM03B-SRSS-TB(LF)(SN)(P), U6 10155435-00011LF, U7 CYW43439KUBGT, X1 TXM12M0004252FBCEO00T

Commit message: main_pcb
Parts:
- removed Q1: DMG1012T-7, footprint:SOT-523-3_L1.6-W0.8-P1.00-LS1.6-BR, symbol DMG1012T-7:DMG1012T-7
- removed R20: 10K, symbol Device:R_Small
- removed R21: 20K, symbol Device:R_Small
- removed SW1, SW2: SW_Push, footprint:SW-SMD_4P-L6.0-W6.0-P4.50-LS7.2, symbol Switch:SW_Push
- removed U7: CYW43439KUBGT, footprint:WLBGA-63_L4.8-W2.8-P0.40-BL_CYW43438KUBGT, symbol CYW43439KUBGT:CYW43439KUBGT
- added D1, D2: Green, LED_SMD:LED_0603_1608Metric_Pad1.05x0.95mm_HandSolder, symbol Device:LED
- added D3: D_Schottky, Diode_SMD:D_SOD-123, symbol Device:D_Schottky
- added F1: 0603L020/30XR, footprint:F0603, symbol 0603L020/30XR:0603L020/30XR
- added L2: 2.2uH, Inductor_SMD:L_APV_ANR6028, symbol Device:L_Small
- added R22, R23: 470R, Resistor_SMD:R_0603_1608Metric_Pad0.98x0.95mm_HandSolder, symbol Device:R_Small
- added R24: 120K, Resistor_SMD:R_0603_1608Metric_Pad0.98x0.95mm_HandSolder, symbol Device:R_Small
- added R25: 100K, Resistor_SMD:R_0603_1608Metric_Pad0.98x0.95mm_HandSolder, symbol Device:R_Small
- added SW3, SW4: SW_Push_Dual, footprint:SW-SMD_4P-L6.0-W6.0-P4.50-LS7.2, symbol Switch:SW_Push_Dual
- added U7: Radio Module 2, footprint:rpi_rmc20452t, symbol RPI_RMC20452T:RPI_RMC20452T
- added U8: TLV62569DBVR, footprint:SOT-23-5_L3.0-W1.7-P0.95-LS2.8-BR, symbol TLV62569DBVR:TLV62569DBVR
- C1, C10, C11, C12, C13, C16, C2, C20, C3, C4, C5, C6, C7, C8, C9: footprint (none) -> Capacitor_SMD:C_0603_1608Metric_Pad1.08x0.95mm_HandSolder
- C14, C15: footprint (none) -> Capacitor_SMD:C_0805_2012Metric_Pad1.18x1.45mm_HandSolder
- C17, C18: footprint (none) -> Capacitor_SMD:C_0402_1005Metric_Pad0.74x0.62mm_HandSolder
- C19: value 2.2uF -> 10uF; footprint (none) -> Capacitor_SMD:C_0805_2012Metric_Pad1.18x1.45mm_HandSolder
- L1: value 3.3u -> 3.3uH; footprint (none) -> footprint:IND-SMD_L2.0-W1.6_AOTA-B201610S3R3-101-T
- R1, R10, R11, R12, R13, R14, R15, R16, R17, R2, R3, R4, R5, R6, R7, R8, R9: footprint (none) -> Resistor_SMD:R_0603_1608Metric_Pad0.98x0.95mm_HandSolder
- R18: value 470R -> 10k; footprint (none) -> Resistor_SMD:R_0603_1608Metric_Pad0.98x0.95mm_HandSolder
- R19: value 10K -> 10k; footprint (none) -> Resistor_SMD:R_0603_1608Metric_Pad0.98x0.95mm_HandSolder
Connections:
- net +1V1: now also C19.1, L2.2, R24.2, R25.1, R25.2, U8.5 (FB)
- net +3V3: now also U7.14 (VDDIO), U7.16 (VIN)
- net GND: now also C19.2, D1.1 (K), D2.1 (K), R24.1, SW3.1, SW3.3, U7.1 (GND), U7.11 (GND), U7.15 (GND), U7.21 (GND), U7.4 (GND), U7.7 (GND), U8.2 (GND); no longer C19.1
- net RUN: now also SW4.2, SW4.4
- net VBUS: now also D3.2 (A), U8.1 (EN), U8.4 (VIN)
- net at R19.1: now also U7.10 (nIRQ)
- net GPIO24: now reaches R18.1
- net GPIO24: now also R19.2, U1.36 (GPIO24), U7.5 (DI)
- net at R15.2: now also SW3.2, SW3.4
- net at R17.1: now also SW4.1, SW4.3
- net +5V: no longer names the net of U2.18 (+5V_Power)
- net +5V: now also C20.1, F1.1
- net GPI7 renamed GPIO7
- net GPIO0: no longer names the net of U1.2 (GPIO0)
- net GPIO0: now also R23.1
- removed net VOUT_CORE: C19.2, C20.1
- net WL_CLK renamed GPIO29_ADC3
- net GPIO29_ADC3: now also U7.3 (SCLK)
- net WL_CS renamed GPIO25
- net GPIO25: now also U7.9 (CS)
- removed net WL_D: R18.2, R19.2, U1.36 (GPIO24)
- net WL_ON renamed GPIO23
- net GPIO23: now also U7.12 (WL_ON), U7.13 (BT_ON)
- new net: L2.1, U8.3 (SW)
- new net: R22.1, U7.8 (GPIO0)
- new net: D1.2 (A), R22.2
- new net: R18.2, U7.6 (DO)
- new net: D2.2 (A), R23.2
- new net: D3.1 (K), F1.2
- no-connect marks 18 -> 4
Other:
- note added: "1%"
- note added: "1% 50mW"
- note removed: "0603 10% 6.3V X5R"
- note removed: "0603 50m W1%"
- note removed: "50mW 1% 0603"
- moved on the sheet: C1, C10, C11, C12, C13, C14, C15, C16, C17, C18, C2, C3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

Commit message: upd
Parts:
- added H1, H2, H3, H4: MountingHole, MountingHole:MountingHole_2.5mm, symbol Mechanical:MountingHole

Commit message: upd
Other:
- moved on the sheet: C14, C15, C16, C17, C18, C19, C20, D1, D3, F1, H1, H2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
